File: KiCad/Console/Console.kicad_sch (KiCad schematic)
At the start: 7 parts, among them J1 Conn_01x10_Pin, J2 Conn_01x08_Pin, J3 Conn_01x08_Pin, J4 Conn_01x06_Pin, J5 Conn_01x06, SW1 RotaryEncoder_Switch, U1 OLED SSD1306 128X64

Commit message: measurement after re-solder
Connections:
- net 3.3V: no longer U1.2 (VCC)
- net 5V: now also U1.2 (VCC)
Changed lines of the file:
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@@
 (kicad_sch (version 20230121) (generator eeschema)
   (paper "A4")
+  (junction (at 81.28 78.74) (diameter 0) (color 0 0 0 0)
+  )
   (junction (at 83.82 135.89) (diameter 0) (color 0 0 0 0)
   )
@@
   )
   (wire (pts (xy 134.62 82.55) (xy 140.97 82.55))
+    (stroke (width 0) (type default))
+  )
+  (wire (pts (xy 81.28 78.74) (xy 99.06 78.74))
     (stroke (width 0) (type default))
   )
@@
     (stroke (width 0) (type default))
   )
-  (wire (pts (xy 63.5 40.64) (xy 63.5 72.39))
+  (wire (pts (xy 81.28 78.74) (xy 81.28 143.51))
     (stroke (width 0) (type default))
   )
-  (wire (pts (xy 99.06 78.74) (xy 78.74 78.74))
+  (wire (pts (xy 63.5 40.64) (xy 63.5 72.39))
     (stroke (width 0) (type default))
   )
@@
     (stroke (width 0) (type default))
   )
-  (wire (pts (xy 81.28 60.96) (xy 81.28 143.51))
+  (wire (pts (xy 81.28 60.96) (xy 81.28 78.74))
     (stroke (width 0) (type default))
   )
@@
     (stroke (width 0) (type default))
   )
-  (wire (pts (xy 78.74 78.74) (xy 78.74 143.51))
-    (stroke (width 0) (type default))
-  )

Commit message: 測定フォルダ更新。
Parts:
- added U2: TSOP4838(?), OptoDevice:Vishay_MOLD-3Pin, symbol Interface_Optical:TSOP41xx
- added U3: TSOP7000, OptoDevice:Vishay_MOLD-3Pin, symbol Interface_Optical:TSOP41xx
Connections:
- net D0: now also U2.1 (OUT)
- net D1: now also U3.1 (OUT)
- net GND: now also U2.2 (GND), U3.2 (GND)
- net 5V renamed +5V
- net +5V: now also U2.3 (Vs), U3.3 (Vs)
Other:
- moved on the sheet: J1, J2, J3, J4, J5, SW1, U1
