File: KiCad/VolumeControlSheild/VolumeControlSheild.kicad_sch (KiCad schematic)
At the start: 16 parts, among them J1 Power, J2 Digital/PWM, J3 Analog, J4 Digital/PWM, J5 Conn_01x08, SW1 EC11E15204A3, U1 TSOP4838(?), U2 TSOP7000, U3 OLED SSH1106, U4 LM317_TO-252

Commit message: Gerber generated.
Parts:
- removed SW1: EC11E15204A3, myfootprint:EC11E15204A3, symbol LogAttSheild:RotaryEncoder_Switch
- added SW1: EC11E15204A3, myfootprint:EC11E15204A3, symbol VolumeControlSheild:RotaryEncoder_Switch
Connections:
- net *3: now also SW1.A1 (A)
- net 2: now also SW1.B1 (B)
- net 7: now also SW1.D1 (S1)
- net GND: now also SW1.C1 (C), SW1.D2 (S2)
